File: Leucht-Ohrringe.kicad_sch (KiCad schematic)
At the start: 14 parts, among them J1 Conn_ARM_SWD_TagConnect_TC2030, P1 USB_C_Plug_USB2.0, U4 CH340N, U5 nRF52832-QFxx

Commit message: add smd antenna, change usb to uart ic to smaller packag
Parts:
- added AE1: Antenna_Chip, Package_TO_SOT_SMD:RFANT3216120A5T, symbol Device:Antenna_Chip
- added C4: 0, Capacitor_SMD:C_0402_1005Metric, symbol Device:C
- added L1: 0, Capacitor_SMD:C_0402_1005Metric, symbol Device:L
- added R2: 0, Capacitor_SMD:C_0402_1005Metric, symbol Device:R
- D2: value ESD411 -> ESD5Z6.0; footprint Button_Switch_SMD:ESD411 -> Diode_SMD:D_SOD-523; LCSC (none) -> C49437732
- D3, D4: value ESD321 -> H4V5HD3UA; footprint Diode_SMD:D_SOD-523 -> Diode_SMD:D_SOD-323; LCSC (none) -> C54334010
Connections:
- net GND: now also R2.1
- net at U5.30 (ANT): now also C4.1
- new net: C4.2, L1.1, R2.2
- new net: AE1.1 (FEED), L1.2

Commit message: add gerbers, fix reversed esd diodes
Parts:
- AE1: LCSC (none) -> C127629
Connections:
- net +5V: now also D2.1 (K); no longer D2.2 (A)
- net D+: now also D3.1 (K); no longer D3.2 (A)
- net D-: now also D4.1 (K); no longer D4.2 (A)
- net GND: now also D2.2 (A), D3.2 (A), D4.2 (A); no longer D2.1 (K), D3.1 (K), D4.1 (K)
