File: Leucht-Ohrringe.kicad_pcb (KiCad board)
At the start: 2 copper layers, 20 x 49.5 mm, 63 parts, among them J1 Conn_ARM_SWD_TagConnect_TC2030, P1 USB_C_Plug_USB2.0, SW1 SW_SPDT, U1 TX4204, U3 ICM-42670-L, U4 CH340N, U5 nRF52832-QFxx

Commit message: update layout
Routing:
- net GND: vias 80 -> 83
